File: board/encoder-port.sch (KiCad schematic (older format))
At the start: 4 parts

Commit message: WIP
Parts:
- J3: renamed from J?; footprint (none) -> Pin_Headers:Pin_Header_Straight_1x05_Pitch2.54mm
- R2, R3, R4: renamed from R?; footprint (none) -> Resistors_SMD:R_0805
Changed lines of the file:
@@
 $Descr A4 11693 8268
 encoding utf-8
-Sheet 2 5
+Sheet 2 16
 Title ""
 Date ""
@@
 $EndDescr
 $Comp
-L Conn_01x05 J?
+L Conn_01x05 J3
 U 1 1 5C26BCAE
 P 5750 2600
-F 0 "J?" H 5750 2900 50  0000 C CNN
+AR Path="/5C26BC0F/5C26BCAE" Ref="J3"  Part="1"
+AR Path="/5C2702EF/5C26BCAE" Ref="J4"  Part="1"
+AR Path="/5C270598/5C26BCAE" Ref="J5"  Part="1"
+AR Path="/5C275CC7/5C26BCAE" Ref="J13"  Part="1"
+F 0 "J3" H 5750 2900 50  0000 C CNN
 F 1 "Encoder" H 6000 2650 50  0000 C CNN
-F 2 "" H 5750 2600 50  0001 C CNN
+F 2 "Pin_Headers:Pin_Header_Straight_1x05_Pitch2.54mm" H 5750 2600 50  0001 C CNN
 F 3 "" H 5750 2600 50  0001 C CNN
 	1    5750 2600
@@
 $EndComp
 $Comp
-L R R?
+L R R4
 U 1 1 5C26BD7D
 P 5400 2200
-F 0 "R?" H 5500 2250 50  0000 C CNN
+AR Path="/5C26BC0F/5C26BD7D" Ref="R4"  Part="1"
+AR Path="/5C2702EF/5C26BD7D" Ref="R7"  Part="1"
+AR Path="/5C270598/5C26BD7D" Ref="R10"  Part="1"
+AR Path="/5C275CC7/5C26BD7D" Ref="R20"  Part="1"
+F 0 "R4" H 5500 2250 50  0000 C CNN
 F 1 "10k" H 5550 2150 50  0000 C CNN
-F 2 "" V 5330 2200 50  0001 C CNN
+F 2 "Resistors_SMD:R_0805" V 5330 2200 50  0001 C CNN
 F 3 "" H 5400 2200 50  0001 C CNN
 	1    5400 2200
@@
 $EndComp
 $Comp
-L R R?
+L R R3
 U 1 1 5C26BE29
 P 5100 2200
-F 0 "R?" H 5200 2250 50  0000 C CNN
+AR Path="/5C26BC0F/5C26BE29" Ref="R3"  Part="1"
+AR Path="/5C2702EF/5C26BE29" Ref="R6"  Part="1"
+AR Path="/5C270598/5C26BE29" Ref="R9"  Part="1"
+AR Path="/5C275CC7/5C26BE29" Ref="R19"  Part="1"
+F 0 "R3" H 5200 2250 50  0000 C CNN
 F 1 "10k" H 5250 2150 50  0000 C CNN
-F 2 "" V 5030 2200 50  0001 C CNN
+F 2 "Resistors_SMD:R_0805" V 5030 2200 50  0001 C CNN
 F 3 "" H 5100 2200 50  0001 C CNN
 	1    5100 2200
@@
 $EndComp
 $Comp
-L R R?
+L R R2
 U 1 1 5C26BE4A
 P 4800 2200
-F 0 "R?" H 4900 2250 50  0000 C CNN
+AR Path="/5C26BC0F/5C26BE4A" Ref="R2"  Part="1"
+AR Path="/5C2702EF/5C26BE4A" Ref="R5"  Part="1"
+AR Path="/5C270598/5C26BE4A" Ref="R8"  Part="1"
+AR Path="/5C275CC7/5C26BE4A" Ref="R18"  Part="1"
+F 0 "R2" H 4900 2250 50  0000 C CNN
 F 1 "10k" H 4950 2150 50  0000 C CNN
-F 2 "" V 4730 2200 50  0001 C CNN
+F 2 "Resistors_SMD:R_0805" V 4730 2200 50  0001 C CNN
 F 3 "" H 4800 2200 50  0001 C CNN
 	1    4800 2200
@@
 $EndComp
 $Comp
-L +3V3 #PWR?
+L +3V3 #PWR021
 U 1 1 5C26BE8C
 P 5450 2700
-F 0 "#PWR?" H 5450 2550 50  0001 C CNN
+AR Path="/5C26BC0F/5C26BE8C" Ref="#PWR021"  Part="1"
+AR Path="/5C2702EF/5C26BE8C" Ref="#PWR026"  Part="1"
+AR Path="/5C270598/5C26BE8C" Ref="#PWR031"  Part="1"
+AR Path="/5C275CC7/5C26BE8C" Ref="#PWR050"  Part="1"
+F 0 "#PWR021" H 5450 2550 50  0001 C CNN
 F 1 "+3V3" H 5450 2840 50  0000 C CNN
 F 2 "" H 5450 2700 50  0001 C CNN
@@
 $EndComp
 $Comp
-L +3V3 #PWR?
+L +3V3 #PWR022
 U 1 1 5C26BEAE
 P 4800 2050
-F 0 "#PWR?" H 4800 1900 50  0001 C CNN
+AR Path="/5C26BC0F/5C26BEAE" Ref="#PWR022"  Part="1"
+AR Path="/5C2702EF/5C26BEAE" Ref="#PWR027"  Part="1"
+AR Path="/5C270598/5C26BEAE" Ref="#PWR032"  Part="1"
+AR Path="/5C275CC7/5C26BEAE" Ref="#PWR051"  Part="1"
+F 0 "#PWR022" H 4800 1900 50  0001 C CNN
 F 1 "+3V3" H 4800 2190 50  0000 C CNN
 F 2 "" H 4800 2050 50  0001 C CNN
@@
 $EndComp
 $Comp
-L +3V3 #PWR?
+L +3V3 #PWR023
 U 1 1 5C26BEE1
 P 5100 2050
-F 0 "#PWR?" H 5100 1900 50  0001 C CNN
+AR Path="/5C26BC0F/5C26BEE1" Ref="#PWR023"  Part="1"
+AR Path="/5C2702EF/5C26BEE1" Ref="#PWR028"  Part="1"
+AR Path="/5C270598/5C26BEE1" Ref="#PWR033"  Part="1"
+AR Path="/5C275CC7/5C26BEE1" Ref="#PWR052"  Part="1"
+F 0 "#PWR023" H 5100 1900 50  0001 C CNN
 F 1 "+3V3" H 5100 2190 50  0000 C CNN
 F 2 "" H 5100 2050 50  0001 C CNN
@@
 $EndComp
 $Comp
-L +3V3 #PWR?
+L +3V3 #PWR024
 U 1 1 5C26BEF8
 P 5400 2050
-F 0 "#PWR?" H 5400 1900 50  0001 C CNN
+AR Path="/5C26BC0F/5C26BEF8" Ref="#PWR024"  Part="1"
+AR Path="/5C2702EF/5C26BEF8" Ref="#PWR029"  Part="1"
+AR Path="/5C270598/5C26BEF8" Ref="#PWR034"  Part="1"
+AR Path="/5C275CC7/5C26BEF8" Ref="#PWR053"  Part="1"
+F 0 "#PWR024" H 5400 1900 50  0001 C CNN
 F 1 "+3V3" H 5400 2190 50  0000 C CNN
 F 2 "" H 5400 2050 50  0001 C CNN
@@
 $EndComp
 $Comp
-L GND #PWR?
+L GND #PWR025
 U 1 1 5C26BF31
 P 5450 2800
-F 0 "#PWR?" H 5450 2550 50  0001 C CNN
+AR Path="/5C26BC0F/5C26BF31" Ref="#PWR025"  Part="1"
+AR Path="/5C2702EF/5C26BF31" Ref="#PWR030"  Part="1"
+AR Path="/5C270598/5C26BF31" Ref="#PWR035"  Part="1"
+AR Path="/5C275CC7/5C26BF31" Ref="#PWR054"  Part="1"
+F 0 "#PWR025" H 5450 2550 50  0001 C CNN
 F 1 "GND" H 5450 2650 50  0000 C CNN
 F 2 "" H 5450 2800 50  0001 C CNN
