File: board/retradio.sch (KiCad schematic (older format))
At the start: 25 parts

Commit message: WIP
Parts:
- C1, C12, C13, C14, C15, C16, C17, C2, C3, C4, C6, C7, C8, C9: renamed from C?; footprint (none) -> Capacitors_SMD:C_0805
- C10, C5: renamed from C?; footprint (none) -> Capacitors_SMD:CP_Elec_8x10
- C11: renamed from C?; value 1000u/6.3V -> 470u/16V; footprint (none) -> Capacitors_SMD:CP_Elec_8x10
- J1, J2: renamed from J?; footprint (none) -> Pin_Headers:Pin_Header_Straight_1x02_Pitch2.54mm
- L1, L2: renamed from L?; footprint (none) -> Inductors_SMD:L_0805
- M1: renamed from M?; footprint (none) -> device.farm:Orange-Pi-Zero
- R1: renamed from R?; footprint (none) -> Resistors_SMD:R_0805
- U2: renamed from U?; footprint MODULE -> Housings_SOIC:SOIC-16_3.9x9.9mm_Pitch1.27mm
- gave numbers to parts that had none: 1

Commit message: WIP
Parts:
- added X1: I2C-6P, Connectors:IDC_Header_Straight_6pins, symbol I2C-6P
- J1, J2: footprint Pin_Headers:Pin_Header_Straight_1x02_Pitch2.54mm -> device.farm:DG301-5.0-02
Connections:
- net +3V3: now also X1.4 (3V3)
- net +5V: now also X1.5 (5V)
- net GND: now also X1.1 (GND)
- net AVCC: now reaches C16.2, C17.2, R1.2, U2.13 (AVCC)
- net VCLAMP: now reaches C3.1, U2.7 (VCLAMP)
- net at C14.1, L1.2: now also J2.2 (Pin_2); no longer J2.1 (Pin_1)
- net at C15.2, L2.2: now also J2.1 (Pin_1); no longer J2.2 (Pin_2)
- net BTN1 renamed SDA
- net SDA: now also X1.3 (SDA)
- net BTN2 renamed SCL
- net SCL: now also X1.2 (SCL)
- net BTN3: no longer names the net of M1.16 (TWI1-SDA/PA19/GPIO19)
- net BTN4: no longer names the net of M1.18 (TWI1-SCK/PA18/GPIO18)
- net BTN5: no longer names the net of M1.7 (PWM1/PA06/GPIO6)
- net EN1_CL renamed ALERT
- net ALERT: now also X1.6 (ALERT)
- net EN1_DT: no longer names the net of M1.10 (UART1_RX/PG07/GPIO199)
- net EN1_SW: no longer names the net of M1.11 (UART2_RX/PA01/GPIO1)
- net EN2_CL: no longer names the net of M1.13 (UART2_TX/PA00/GPIO0)
- net EN2_DT: no longer names the net of M1.15 (UART2_CTS/PA03/GPIO3)
- net EN2_SW: no longer names the net of M1.19 (SPI1_MOSI/PA15/GPIO15)
- net EN3_CL: no longer names the net of M1.21 (SPI1_MISO/PA16/GPIO16)
- net EN3_DT: no longer names the net of M1.22 (UART2_RTS/PA02/GPIO2)
- net EN3_SW: no longer names the net of M1.23 (SPI1_CLK/PA14/GPIO14)
- net EN4_CL: no longer names the net of M1.24 (SPI1_CS/PA13/GPIO13)
- net EN4_DT: no longer names the net of M1.26 (SIM_DET/PA_EINT10/PA10/GPIO10)
- net EN4_SW: no longer names the net of M1.12 (SIM_CLK/PA_EINT7/PA07/GPIO7)
- no-connect marks 12 -> 26
