File: board/retradio.kicad_pcb (KiCad board)
At the start: 2 copper layers, 63 parts, among them J1 Power, J10 Button, J11 Button, J12 Button, J13 Encoder, J14 LED, J15 LED, J16 LED, J17 LED, J2 Speaker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

Commit message: WIP
Parts:
- M1: moved to B.Cu
- moved J2 115.3 mm to (95.1, 71.7)
- moved C16 101.4 mm to (104.0, 76.0)
- moved C14 101.0 mm to (104.0, 85.0)
- moved R1 100.5 mm to (104.0, 73.0)
- moved C17 100.0 mm to (104.0, 70.0)
- moved L1 99.4 mm to (104.0, 82.0), turned to 180 degrees
- moved C15 97.4 mm to (104.0, 61.0), turned to 180 degrees
- moved C12 97.3 mm to (104.0, 79.0), turned to 180 degrees
- moved L2 96.8 mm to (104.0, 64.0), turned to 180 degrees
- moved C13 95.5 mm to (104.0, 67.0), turned to 180 degrees
- moved C9 86.4 mm to (109.0, 83.0)
- moved C8 84.3 mm to (109.0, 80.0), turned to 0 degrees
- moved C6 82.7 mm to (109.0, 63.0), turned to 0 degrees
- moved C10 81.8 mm to (117.0, 84.0)
- moved C7 81.8 mm to (109.0, 66.0), turned to 0 degrees
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Other:
- board outline added: 48 x 64 mm

Commit message: WIP
Parts:
- removed J10, J11, J12, J6, J7, J8, J9: Button, Pin_Headers:Pin_Header_Straight_1x02_Pitch2.54mm
- removed J13, J3, J4, J5: Encoder, Pin_Headers:Pin_Header_Straight_1x05_Pitch2.54mm
- removed J14, J15, J16, J17: LED, Pin_Headers:Pin_Header_Straight_1x02_Pitch2.54mm
- removed R10, R11, R12, R13, R14, R15, R16, R17, R18, R19, R2, R20, R3, R4, R5, R6, R7, R8, R9: 10k, Resistors_SMD:R_0805
- removed R21, R22, R23, R24: 270R, Resistors_SMD:R_0805
- added X1: I2C-6P, Connectors:IDC_Header_Straight_6pins, F.Cu at (95.0, 61.0)
- J1, J2: footprint Pin_Headers:Pin_Header_Straight_1x02_Pitch2.54mm -> device.farm:DG301-5.0-02
- moved U1 72.9 mm to (112.3, 45.0)
- moved C4 70.3 mm to (106.0, 45.0), turned to 270 degrees
- moved J1 65.5 mm to (100.5, 45.0), turned to 180 degrees
- moved C11 8.55 mm to (123.5, 45.0)
- moved J2 5.61 mm to (97.0, 77.0), turned to 270 degrees
Connections:
- net Net-(C16-Pad2) renamed /AVCC
- net Net-(C3-Pad1) renamed /VCLAMP
- J2 pad 1: Net-(C14-Pad1) -> Net-(C15-Pad2)
- J2 pad 2: Net-(C15-Pad2) -> Net-(C14-Pad1)
- M1 pad 10: /EN1_DT -> (no net)
- M1 pad 11: /EN1_SW -> (no net)
- M1 pad 13: /EN2_CL -> (no net)
- M1 pad 15: /EN2_DT -> (no net)
- M1 pad 16: /BTN3 -> (no net)
- M1 pad 18: /BTN4 -> (no net)
- M1 pad 19: /EN2_SW -> (no net)
- M1 pad 21: /EN3_CL -> (no net)
- M1 pad 22: /EN3_DT -> (no net)
- M1 pad 23: /EN3_SW -> (no net)
- M1 pad 24: /EN4_CL -> (no net)
- M1 pad 26: /EN4_DT -> (no net)
- M1 pad 3: /BTN1 -> /SDA
- M1 pad 5: /BTN2 -> /SCL
- M1 pad 7: /BTN5 -> (no net)
- M1 pad 8: /EN1_CL -> /ALERT
Other:
- board size 48 x 64 mm -> 39 x 56 mm

Commit message: WIP
Routing:
- net +12V: track 0.00 -> 143.7 mm
- net +5V: track 0.00 -> 82.8 mm
- net GND: track 0.00 -> 67.6 mm, vias 0 -> 13
- net +3V3: track 0.00 -> 65.0 mm, vias 0 -> 2
- net /SCL: track 0.00 -> 44.0 mm
- net /ALERT: track 0.00 -> 40.5 mm, vias 0 -> 1
- net /SDA: track 0.00 -> 38.6 mm
- net /AUDIO: track 0.00 -> 26.9 mm
- net Net-(C15-Pad2): track 0.00 -> 18.5 mm
- net /AVCC: track 0.00 -> 10.7 mm
- net Net-(C14-Pad1): track 0.00 -> 9.07 mm
- net Net-(C13-Pad1): track 0.00 -> 8.56 mm
- net Net-(C12-Pad1): track 0.00 -> 8.56 mm
- net Net-(C13-Pad2): track 0.00 -> 8.07 mm
- net Net-(C12-Pad2): track 0.00 -> 8.07 mm
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- added copper zone on B.Cu, net GND
Other:
- net class Default: trace_width 0.25 -> 0.4
- net class PWR added: clearance 0.2, trace_width 1, via_dia 1, via_drill 0.8
- board text added: "+12V"
- board text added: "GND"
- board text added: "I2C"
- board text added: "RETRADIO v1.0"
- board text added: "SPEAKER"
