File: mb-a/mb-a.kicad_pcb (KiCad board)
At the start: 2 copper layers, 39 x 56 mm, 26 parts, among them J1 Power, J2 Speaker, M1 Orange-Pi-Zero, U1 NCP1117-5.0_SOT223, U2 PAM8320, X1 I2C-6P

Commit message: WIP
Parts:
- added R2: 1k5, Resistors_SMD:R_0805, F.Cu at (108.0, 57.0)
- added R3: 1k5, Resistors_SMD:R_0805, F.Cu at (105.0, 57.0)
- added R4: 1k5, Resistors_SMD:R_0805, F.Cu at (102.5, 57.0)
Routing:
- net +3V3: track 65.0 -> 82.3 mm
- net /SDA: track 38.6 -> 53.9 mm
- net /ALERT: track 40.5 -> 53.5 mm
- net +12V: track 143.7 -> 153.2 mm
- net /SCL: track 44.0 -> 51.4 mm
Other:
- board text added: "RR-MB-A v1.0"
- board text removed: "RETRADIO v1.0"

Commit message: WIP
Connections:
- U2 pad 12: (no net) -> GND
- U2 pad 2: (no net) -> /AVCC
Routing:
- net +5V: track 82.8 -> 101.8 mm, vias 0 -> 1
- net /AVCC: track 10.7 -> 20.9 mm, vias 0 -> 2
- net GND: track 67.6 -> 70.7 mm
Other:
- board text added: "RR-MB-A v1.1"
- board text removed: "RR-MB-A v1.0"
