File: mb-a/mb-a.kicad_pcb (KiCad board)
At the start: 2 copper layers, 39 x 56 mm, 29 parts, among them J1 Power, J2 Speaker, M1 Orange-Pi-Zero, U1 NCP1117-5.0_SOT223, U2 PAM8320, X1 I2C-6P

Commit message: WIP
Parts:
- C1, C12, C13, C14, C15, C16, C17, C2, C3, C4, C6, C7, C8, C9: footprint Capacitors_SMD:C_0805 -> Capacitor_SMD:C_0805_2012Metric
- C10, C11, C5: footprint Capacitors_SMD:CP_Elec_8x10 -> Capacitor_SMD:CP_Elec_8x10
- L1, L2: footprint Inductors_SMD:L_0805 -> Inductor_SMD:L_0805_2012Metric
- R1, R2, R3, R4: footprint Resistors_SMD:R_0805 -> Resistor_SMD:R_0805_2012Metric
- U1: footprint TO_SOT_Packages_SMD:SOT-223-3Lead_TabPin2 -> Package_TO_SOT_SMD:SOT-223-3_TabPin2
- U2: footprint Housings_SOIC:SOIC-16_3.9x9.9mm_Pitch1.27mm -> Package_SO:SOIC-16_3.9x9.9mm_P1.27mm
- X1: footprint Connectors:IDC_Header_Straight_6pins -> Connector_IDC:IDC-Header_2x03_P2.54mm_Vertical
- moved X1 0.08 mm to (95.0, 60.9), turned to 0 degrees
Connections:
- M1 pad 10: (no net) -> Net-(M1-Pad10)
- M1 pad 11: (no net) -> Net-(M1-Pad11)
- M1 pad 12: (no net) -> Net-(M1-Pad12)
- M1 pad 13: (no net) -> Net-(M1-Pad13)
- M1 pad 15: (no net) -> Net-(M1-Pad15)
- M1 pad 16: (no net) -> Net-(M1-Pad16)
- M1 pad 18: (no net) -> Net-(M1-Pad18)
- M1 pad 19: (no net) -> Net-(M1-Pad19)
- M1 pad 21: (no net) -> Net-(M1-Pad21)
- M1 pad 22: (no net) -> Net-(M1-Pad22)
- M1 pad 23: (no net) -> Net-(M1-Pad23)
- M1 pad 24: (no net) -> Net-(M1-Pad24)
- M1 pad 26: (no net) -> Net-(M1-Pad26)
- M1 pad 29: (no net) -> Net-(M1-Pad29)
- M1 pad 30: (no net) -> Net-(M1-Pad30)
- M1 pad 31: (no net) -> Net-(M1-Pad31)
- M1 pad 32: (no net) -> Net-(M1-Pad32)
- M1 pad 34: (no net) -> Net-(M1-Pad34)
- M1 pad 35: (no net) -> Net-(M1-Pad35)
- M1 pad 36: (no net) -> Net-(M1-Pad36)
- M1 pad 37: (no net) -> Net-(M1-Pad37)
- M1 pad 38: (no net) -> Net-(M1-Pad38)
- M1 pad 39: (no net) -> Net-(M1-Pad39)
- M1 pad 7: (no net) -> Net-(M1-Pad7)

Commit message: WIP
Parts:
- added C18: 100n, Capacitor_SMD:C_0805_2012Metric, F.Cu at (120.5, 46.7)
- added C19: 100u/12V, Capacitor_SMD:CP_Elec_6.3x5.4, B.Cu at (126.5, 44.5)
- added L3: 6.8uH, mb-a:L_Taiyo-Yuden_NR-60xx_HandSoldering, B.Cu at (116.5, 45.5)
- added R5: 100k, Resistor_SMD:R_0805_2012Metric, F.Cu at (115.1, 43.2)
- added R6: 30.9k 1%, Resistor_SMD:R_0805_2012Metric, F.Cu at (124.5, 43.2)
- added R7: 4.22k 1%, Resistor_SMD:R_0805_2012Metric, F.Cu at (122.1, 43.2)
- C11: value 470u/16V -> 100n; footprint Capacitor_SMD:CP_Elec_8x10 -> Capacitor_SMD:C_0805_2012Metric
- C4: value 10u -> 100u/12V; footprint Capacitor_SMD:C_0805_2012Metric -> Capacitor_SMD:CP_Elec_6.3x5.4; moved to B.Cu
- U1: value NCP1117-5.0_SOT223 -> FR8205; footprint Package_TO_SOT_SMD:SOT-223-3_TabPin2 -> Package_TO_SOT_SMD:SOT-23-6
- moved C11 11.0 mm to (112.6, 43.2), turned to 270 degrees
- moved U1 6.51 mm to (118.6, 43.3), turned to 180 degrees
- moved C4 0.71 mm to (106.5, 44.5), turned to 90 degrees
Connections:
- C11 pad 1: +5V -> GND
- C11 pad 2: GND -> +12V
- C4 pad 1: GND -> +12V
- C4 pad 2: +12V -> GND
- M1 pad 10: Net-(M1-Pad10) -> (no net)
- M1 pad 11: Net-(M1-Pad11) -> (no net)
- M1 pad 12: Net-(M1-Pad12) -> (no net)
- M1 pad 13: Net-(M1-Pad13) -> (no net)
- M1 pad 15: Net-(M1-Pad15) -> (no net)
- M1 pad 16: Net-(M1-Pad16) -> (no net)
- M1 pad 18: Net-(M1-Pad18) -> (no net)
- M1 pad 19: Net-(M1-Pad19) -> (no net)
- M1 pad 21: Net-(M1-Pad21) -> (no net)
- M1 pad 22: Net-(M1-Pad22) -> (no net)
- M1 pad 23: Net-(M1-Pad23) -> (no net)
- M1 pad 24: Net-(M1-Pad24) -> (no net)
- M1 pad 26: Net-(M1-Pad26) -> (no net)
- M1 pad 29: Net-(M1-Pad29) -> (no net)
- M1 pad 30: Net-(M1-Pad30) -> (no net)
- M1 pad 31: Net-(M1-Pad31) -> (no net)
- M1 pad 32: Net-(M1-Pad32) -> (no net)
- M1 pad 34: Net-(M1-Pad34) -> (no net)
- M1 pad 35: Net-(M1-Pad35) -> (no net)
- M1 pad 36: Net-(M1-Pad36) -> (no net)
- M1 pad 37: Net-(M1-Pad37) -> (no net)
- M1 pad 38: Net-(M1-Pad38) -> (no net)
- M1 pad 39: Net-(M1-Pad39) -> (no net)
- M1 pad 7: Net-(M1-Pad7) -> (no net)
- U1 pad 1: GND -> Net-(C18-Pad1)
- U1 pad 2: +5V -> GND
- U1 pad 3: +12V -> Net-(R6-Pad1)
Routing:
- net +12V: track 153.2 -> 166.7 mm, vias 0 -> 1
- net Net-(C18-Pad2): track 0.00 -> 8.78 mm, vias 0 -> 1
- net Net-(R6-Pad1): track 0.00 -> 4.79 mm
- net Net-(C18-Pad1): track 0.00 -> 3.21 mm
- net GND: track 70.7 -> 67.7 mm
- net +5V: track 101.8 -> 104.6 mm
- net Net-(R5-Pad1): track 0.00 -> 2.42 mm
Other:
- board size 39 x 56 mm -> 39 x 57 mm
- board text added: "RETRADIO-MB-A v1.2"
- board text removed: "RR-MB-A v1.1"
