File: mb-a/mb-a.sch (KiCad schematic (older format))
At the start: 26 parts, among them J1 Power, J2 Speaker, M1 Orange-Pi-Zero, U1 NCP1117-5.0_SOT223, U2 PAM8320, X1 I2C-6P

Commit message: WIP
Parts:
- added R2, R3, R4: 1k5, Resistors_SMD:R_0805, symbol R
Connections:
- net +3V3: now also R2.1, R3.1, R4.1
- net ALERT: now also R2.2
- net SCL: now also R4.2
- net SDA: now also R3.2
Changed lines of the file:
@@
 	0    -1   -1   0
 $EndComp
+$Comp
+L R R2
+U 1 1 5C2E3068
+P 5450 2050
+F 0 "R2" V 5350 2000 50  0000 C CNN
+F 1 "1k5" V 5350 2150 50  0000 C CNN
+F 2 "Resistors_SMD:R_0805" V 5380 2050 50  0001 C CNN
+F 3 "" H 5450 2050 50  0001 C CNN
+	1    5450 2050
+	0    1    1    0
+$EndComp
+$Comp
+L R R3
+U 1 1 5C2E32B9
+P 5450 2400
+F 0 "R3" V 5350 2350 50  0000 C CNN
+F 1 "1k5" V 5350 2500 50  0000 C CNN
+F 2 "Resistors_SMD:R_0805" V 5380 2400 50  0001 C CNN
+F 3 "" H 5450 2400 50  0001 C CNN
+	1    5450 2400
+	0    1    1    0
+$EndComp
+$Comp
+L R R4
+U 1 1 5C2E3327
+P 5450 2500
+F 0 "R4" V 5550 2450 50  0000 C CNN
+F 1 "1k5" V 5550 2600 50  0000 C CNN
+F 2 "Resistors_SMD:R_0805" V 5380 2500 50  0001 C CNN
+F 3 "" H 5450 2500 50  0001 C CNN
+	1    5450 2500
+	0    1    1    0
+$EndComp
+Wire Wire Line
+	4950 2050 5300 2050
+Wire Wire Line
+	4950 2400 5300 2400
+Wire Wire Line
+	4950 2500 5300 2500
+$Comp
+L +3V3 #PWR034
+U 1 1 5C2E35B7
+P 5600 2050
+F 0 "#PWR034" H 5600 1900 50  0001 C CNN
+F 1 "+3V3" V 5600 2250 50  0000 C CNN
+F 2 "" H 5600 2050 50  0001 C CNN
+F 3 "" H 5600 2050 50  0001 C CNN
+	1    5600 2050
+	0    1    1    0
+$EndComp
+$Comp
+L +3V3 #PWR035
+U 1 1 5C2E3619
+P 5600 2400
+F 0 "#PWR035" H 5600 2250 50  0001 C CNN
+F 1 "+3V3" V 5600 2600 50  0000 C CNN
+F 2 "" H 5600 2400 50  0001 C CNN
+F 3 "" H 5600 2400 50  0001 C CNN
+	1    5600 2400
+	0    1    1    0
+$EndComp
+$Comp
+L +3V3 #PWR036
+U 1 1 5C2E367B
+P 5600 2500
+F 0 "#PWR036" H 5600 2350 50  0001 C CNN
+F 1 "+3V3" V 5600 2700 50  0000 C CNN
+F 2 "" H 5600 2500 50  0001 C CNN
+F 3 "" H 5600 2500 50  0001 C CNN
+	1    5600 2500
+	0    1    1    0
+$EndComp
 $EndSCHEMATC

Commit message: WIP
Connections:
- net AVCC: now also U2.2 (SDN)
- net GND: now also U2.12 (MUTE)
- no-connect marks 26 -> 24
Changed lines of the file:
@@
 LIBS:device.farm
 LIBS:PAM8320
-LIBS:retradio-cache
+LIBS:mb-a-cache
 EELAYER 25 0
 EELAYER END
@@
 	0    -1   -1   0
 $EndComp
-NoConn ~ 2450 5750
-NoConn ~ 3950 6050
 $Comp
 L C C1
@@
 U 1 1 5C2635DF
 P 4250 5850
-F 0 "C12" V 4300 5700 50  0000 L CNN
-F 1 "1u" V 4300 5950 50  0000 L CNN
+F 0 "C12" V 4300 5950 50  0000 L CNN
+F 1 "1u" V 4200 5950 50  0000 L CNN
 F 2 "Capacitors_SMD:C_0805" H 4288 5700 50  0001 C CNN
 F 3 "" H 4250 5850 50  0001 C CNN
@@
 U 1 1 5C263F13
 P 4250 6150
-F 0 "C13" V 4200 6000 50  0000 L CNN
-F 1 "1u" V 4200 6250 50  0000 L CNN
+F 0 "C13" V 4200 6250 50  0000 L CNN
+F 1 "1u" V 4300 6250 50  0000 L CNN
 F 2 "Capacitors_SMD:C_0805" H 4288 6000 50  0001 C CNN
 F 3 "" H 4250 6150 50  0001 C CNN
@@
 Connection ~ 4850 6350
 Wire Wire Line
-	3950 5950 4050 5950
-Wire Wire Line
-	4050 5950 4050 6000
-Wire Wire Line
-	4050 6000 4900 6000
+	3950 5950 4200 5950
+Wire Wire Line
+	4200 5950 4200 6000
+Wire Wire Line
+	4200 6000 4900 6000
 Wire Wire Line
 	5800 5650 5800 5950
@@
 	0    1    1    0
 $EndComp
+$Comp
+L GND #PWR037
+U 1 1 5C548ADA
+P 3950 6050
+F 0 "#PWR037" H 3950 5800 50  0001 C CNN
+F 1 "GND" V 4000 5900 50  0000 C CNN
+F 2 "" H 3950 6050 50  0001 C CNN
+F 3 "" H 3950 6050 50  0001 C CNN
+	1    3950 6050
+	0    -1   -1   0
+$EndComp
+Text Label 2450 5750 2    60   ~ 0
+AVCC
 $EndSCHEMATC

Commit message: WIP
Parts:
- C1, C12, C13, C14, C15, C16, C17, C2, C3, C4, C6, C7, C8, C9: symbol C -> mb-a-rescue:C-mb-a-rescue
- C10, C11, C5: symbol CP -> mb-a-rescue:CP-mb-a-rescue
- J1, J2: symbol Conn_01x02 -> mb-a-rescue:Conn_01x02-mb-a-rescue
- L1, L2: symbol L -> mb-a-rescue:L-mb-a-rescue
- M1: symbol Orange-Pi-Zero -> mb-a-rescue:Orange-Pi-Zero-mb-a-rescue
- R1, R2, R3, R4: symbol R -> mb-a-rescue:R-mb-a-rescue
- U1: symbol NCP1117-5.0_SOT223 -> mb-a-rescue:NCP1117-5.0_SOT223-mb-a-rescue
- U2: symbol PAM8320 -> mb-a-rescue:PAM8320-mb-a-rescue
- X1: symbol I2C-6P -> mb-a-rescue:I2C-6P-mb-a-rescue

Commit message: WIP
Parts:
- C1, C12, C13, C14, C15, C16, C17, C2, C3, C4, C6, C7, C8, C9: footprint Capacitors_SMD:C_0805 -> Capacitor_SMD:C_0805_2012Metric; symbol mb-a-rescue:C-mb-a-rescue -> Device:C
- C10, C11, C5: footprint Capacitors_SMD:CP_Elec_8x10 -> Capacitor_SMD:CP_Elec_8x10; symbol mb-a-rescue:CP-mb-a-rescue -> Device:CP
- J1, J2: symbol mb-a-rescue:Conn_01x02-mb-a-rescue -> Connector_Generic:Conn_01x02
- L1, L2: footprint Inductors_SMD:L_0805 -> Inductor_SMD:L_0805_2012Metric; symbol mb-a-rescue:L-mb-a-rescue -> Device:L
- M1: symbol mb-a-rescue:Orange-Pi-Zero-mb-a-rescue -> device.farm:Orange-Pi-Zero
- R1, R2, R3, R4: footprint Resistors_SMD:R_0805 -> Resistor_SMD:R_0805_2012Metric; symbol mb-a-rescue:R-mb-a-rescue -> Device:R
- U1: footprint TO_SOT_Packages_SMD:SOT-223-3Lead_TabPin2 -> Package_TO_SOT_SMD:SOT-223-3_TabPin2; symbol mb-a-rescue:NCP1117-5.0_SOT223-mb-a-rescue -> Regulator_Linear:NCP1117-5.0_SOT223
- U2: footprint Housings_SOIC:SOIC-16_3.9x9.9mm_Pitch1.27mm -> Package_SO:SOIC-16_3.9x9.9mm_P1.27mm; symbol mb-a-rescue:PAM8320-mb-a-rescue -> PAM8320:PAM8320
- X1: footprint Connectors:IDC_Header_Straight_6pins -> Connector_IDC:IDC-Header_2x03_P2.54mm_Vertical; symbol mb-a-rescue:I2C-6P-mb-a-rescue -> device.farm:I2C-6P

Commit message: WIP
Parts:
- removed C11: 470u/16V, Capacitor_SMD:CP_Elec_8x10, symbol Device:CP
- removed C4: 10u, Capacitor_SMD:C_0805_2012Metric, symbol Device:C
- removed U1: NCP1117-5.0_SOT223, Package_TO_SOT_SMD:SOT-223-3_TabPin2, symbol Regulator_Linear:NCP1117-5.0_SOT223
- added C? (x2): 100u/12V, Capacitor_SMD:CP_Elec_8x10, symbol Device:CP
- added C? (x2): 100n, Capacitor_SMD:C_0805_2012Metric, symbol Device:C
- added L?: 6.8uH, Inductor_SMD:L_0805_2012Metric, symbol Device:L
- added R?: 100k, Resistor_SMD:R_0805_2012Metric, symbol Device:R
- added R?: 30.9k 1%, Resistor_SMD:R_0805_2012Metric, symbol Device:R
- added R?: 4.22k 1%, Resistor_SMD:R_0805_2012Metric, symbol Device:R
- added U?: FR8205, symbol device.farm:FR8205
Connections:
- net +12V: now also C?.1, C?.2, R?.2, U?.5 (VIN)
- net +5V: now also C?.1, L?.2, R?.2
- net GND: now also C?.1, C?.2, C?.2, R?.1, U?.2 (GND)
- new net: C?.1, U?.1 (BST)
- new net: R?.1, R?.2, U?.3 (FB)
- new net: R?.1, U?.4 (SHDN)
- new net: C?.2, L?.1, U?.6 (LX)
Other:
- moved on the sheet: J1, R2, R3, R4, X1

Commit message: WIP
Parts:
- C19, C4: renamed from C?; footprint Capacitor_SMD:CP_Elec_8x10 -> Capacitor_SMD:CP_Elec_6.3x5.4
- L3: renamed from L?; footprint Inductor_SMD:L_0805_2012Metric -> mb-a:L_Taiyo-Yuden_NR-60xx_HandSoldering
- U1: renamed from U?; footprint (none) -> Package_TO_SOT_SMD:SOT-23-6
- gave numbers to parts that had none: 5
Changed lines of the file:
@@
 	8650 4150 8750 4150
 $Comp
-L power:+12V #PWR?
+L power:+12V #PWR013
 U 1 1 5CC2A9BB
 P 2900 1500
-F 0 "#PWR?" H 2900 1350 50  0001 C CNN
+F 0 "#PWR013" H 2900 1350 50  0001 C CNN
 F 1 "+12V" V 2900 1700 50  0000 C CNN
 F 2 "" H 2900 1500 50  0001 C CNN
@@
 $EndComp
 $Comp
-L Device:CP C?
+L Device:CP C4
 U 1 1 5CC2AB6A
 P 3150 1850
-F 0 "C?" H 2950 1950 50  0000 L CNN
+F 0 "C4" H 2950 1950 50  0000 L CNN
 F 1 "100u/12V" H 2750 1750 50  0000 L CNN
-F 2 "Capacitor_SMD:CP_Elec_8x10" H 3188 1700 50  0001 C CNN
+F 2 "Capacitor_SMD:CP_Elec_6.3x5.4" H 3188 1700 50  0001 C CNN
 F 3 "" H 3150 1850 50  0001 C CNN
 	1    3150 1850
@@
 $EndComp
 $Comp
-L Device:C C?
+L Device:C C11
 U 1 1 5CC2AC38
 P 3450 1850
-F 0 "C?" H 3300 1750 50  0000 L CNN
+F 0 "C11" H 3300 1750 50  0000 L CNN
 F 1 "100n" H 3250 1950 50  0000 L CNN
 F 2 "Capacitor_SMD:C_0805_2012Metric" H 3488 1700 50  0001 C CNN
@@
 	3450 1500 3700 1500
 $Comp
-L power:GND #PWR?
+L power:GND #PWR014
 U 1 1 5CC3BDFB
 P 4100 2350
-F 0 "#PWR?" H 4100 2100 50  0001 C CNN
+F 0 "#PWR014" H 4100 2100 50  0001 C CNN
 F 1 "GND" H 4100 2200 50  0000 C CNN
 F 2 "" H 4100 2350 50  0001 C CNN
@@
 $EndComp
 $Comp
-L Device:R R?
+L Device:R R5
 U 1 1 5CC3BF06
 P 3750 1150
-F 0 "R?" V 3650 1050 50  0000 C CNN
+F 0 "R5" V 3650 1050 50  0000 C CNN
 F 1 "100k" V 3650 1250 50  0000 C CNN
 F 2 "Resistor_SMD:R_0805_2012Metric" V 3680 1150 50  0001 C CNN
@@
 $EndComp
 $Comp
-L Device:C C?
+L Device:C C18
 U 1 1 5CC3BFCE
 P 4450 1150
-F 0 "C?" V 4550 1250 50  0000 L CNN
+F 0 "C18" V 4550 1250 50  0000 L CNN
 F 1 "100n" V 4550 900 50  0000 L CNN
 F 2 "Capacitor_SMD:C_0805_2012Metric" H 4488 1000 50  0001 C CNN
@@
 	4650 1150 4600 1150
 $Comp
-L Device:L L?
+L Device:L L3
 U 1 1 5CC48C37
 P 4850 1500
-F 0 "L?" V 4800 1500 50  0000 C CNN
+F 0 "L3" V 4800 1500 50  0000 C CNN
 F 1 "6.8uH" V 4925 1500 50  0000 C CNN
-F 2 "Inductor_SMD:L_0805_2012Metric" H 4850 1500 50  0001 C CNN
+F 2 "mb-a:L_Taiyo-Yuden_NR-60xx_HandSoldering" H 4850 1500 50  0001 C CNN
 F 3 "" H 4850 1500 50  0001 C CNN
 	1    4850 1500
@@
 Connection ~ 4650 1500
 $Comp
-L Device:R R?
+L Device:R R6
 U 1 1 5CC4FC6C
 P 5000 1700
-F 0 "R?" H 4900 1700 50  0000 C CNN
+F 0 "R6" H 4900 1700 50  0000 C CNN
 F 1 "30.9k 1%" H 5250 1700 50  0000 C CNN
 F 2 "Resistor_SMD:R_0805_2012Metric" V 4930 1700 50  0001 C CNN
@@
 $EndComp
 $Comp
-L Device:R R?
+L Device:R R7
 U 1 1 5CC6B922
 P 5000 2100
-F 0 "R?" H 4900 2100 50  0000 C CNN
+F 0 "R7" H 4900 2100 50  0000 C CNN
 F 1 "4.22k 1%" H 5250 2100 50  0000 C CNN
 F 2 "Resistor_SMD:R_0805_2012Metric" V 4930 2100 50  0001 C CNN
@@
 	5000 1550 5000 1500
 $Comp
-L device.farm:FR8205 U?
+L device.farm:FR8205 U1
 U 1 1 5CC26308
 P 4100 1800
-F 0 "U?" H 4400 1350 50  0000 R CNN
+F 0 "U1" H 4400 1350 50  0000 R CNN
 F 1 "FR8205" H 4450 1450 50  0000 R CNN
-F 2 "" H 3400 1250 50  0001 C CNN
+F 2 "Package_TO_SOT_SMD:SOT-23-6" H 3400 1250 50  0001 C CNN
 F 3 "https://datasheet.lcsc.com/szlcsc/FR8205AS6CTR_C172765.pdf" H 3400 1250 50  0001 C CNN
 	1    4100 1800
@@
 	4100 2200 4100 2300
 $Comp
-L Device:CP C?
+L Device:CP C19
 U 1 1 5CC90415
 P 5400 1850
-F 0 "C?" H 5500 1950 50  0000 L CNN
+F 0 "C19" H 5500 1950 50  0000 L CNN
 F 1 "100u/12V" H 5500 1750 50  0000 L CNN
-F 2 "Capacitor_SMD:CP_Elec_8x10" H 5438 1700 50  0001 C CNN
+F 2 "Capacitor_SMD:CP_Elec_6.3x5.4" H 5438 1700 50  0001 C CNN
 F 3 "" H 5400 1850 50  0001 C CNN
 	1    5400 1850
@@
 Connection ~ 5000 2300
 $Comp
-L power:+5V #PWR?
+L power:+5V #PWR015
 U 1 1 5CC9CAD4
 P 5550 1500
-F 0 "#PWR?" H 5550 1350 50  0001 C CNN
+F 0 "#PWR015" H 5550 1350 50  0001 C CNN
 F 1 "+5V" H 5550 1640 50  0000 C CNN
 F 2 "" H 5550 1500 50  0001 C CNN
@@
 	0    1    1    0
 $EndComp
+$Comp
+L power:PWR_FLAG #FLG0101
+U 1 1 5CC267A3
+P 1900 3350
+F 0 "#FLG0101" H 1900 3425 50  0001 C CNN
+F 1 "PWR_FLAG" V 1900 3650 50  0000 C CNN
+F 2 "" H 1900 3350 50  0001 C CNN
+F 3 "" H 1900 3350 50  0001 C CNN
+	1    1900 3350
+	0    -1   -1   0
+$EndComp
+$Comp
+L power:+5V #PWR0101
+U 1 1 5CC268C6
+P 1900 3350
+F 0 "#PWR0101" H 1900 3200 50  0001 C CNN
+F 1 "+5V" V 1900 3550 50  0000 C CNN
+F 2 "" H 1900 3350 50  0001 C CNN
+F 3 "" H 1900 3350 50  0001 C CNN
+	1    1900 3350
+	0    1    1    0
+$EndComp
