File: mb-a/mb-a.sch (KiCad schematic (older format))
At the start: 29 parts, among them J1 Power, J2 Speaker, M1 Orange-Pi-Zero, U1 NCP1117-5.0_SOT223, U2 PAM8320, X1 I2C-6P

Commit message: Band switch support
Parts:
- removed C11: 470u/16V, Capacitors_SMD:CP_Elec_8x10, symbol mb-a-rescue:CP-mb-a-rescue
- removed C4: 10u, Capacitors_SMD:C_0805, symbol mb-a-rescue:C-mb-a-rescue
- removed U1: NCP1117-5.0_SOT223, TO_SOT_Packages_SMD:SOT-223-3Lead_TabPin2, symbol mb-a-rescue:NCP1117-5.0_SOT223-mb-a-rescue
- added C11, C18: 100n, Capacitor_SMD:C_0805_2012Metric, symbol Device:C
- added C19, C4: 100u/12V, Capacitor_SMD:CP_Elec_6.3x5.4, symbol Device:CP
- added L3: 6.8uH, mb-a:L_Taiyo-Yuden_NR-60xx_HandSoldering, symbol Device:L
- added R5: 100k, Resistor_SMD:R_0805_2012Metric, symbol Device:R
- added R6: 30.9k 1%, Resistor_SMD:R_0805_2012Metric, symbol Device:R
- added R7: 4.22k 1%, Resistor_SMD:R_0805_2012Metric, symbol Device:R
- added U1: FR8205, Package_TO_SOT_SMD:SOT-23-6, symbol device.farm:FR8205
- C1, C12, C13, C14, C15, C16, C17, C2, C3, C6, C7, C8, C9: footprint Capacitors_SMD:C_0805 -> Capacitor_SMD:C_0805_2012Metric; symbol mb-a-rescue:C-mb-a-rescue -> Device:C
- C10, C5: footprint Capacitors_SMD:CP_Elec_8x10 -> Capacitor_SMD:CP_Elec_8x10; symbol mb-a-rescue:CP-mb-a-rescue -> Device:CP
- J1, J2: symbol mb-a-rescue:Conn_01x02-mb-a-rescue -> Connector_Generic:Conn_01x02
- L1, L2: footprint Inductors_SMD:L_0805 -> Inductor_SMD:L_0805_2012Metric; symbol mb-a-rescue:L-mb-a-rescue -> Device:L
- M1: symbol mb-a-rescue:Orange-Pi-Zero-mb-a-rescue -> device.farm:Orange-Pi-Zero
- R1, R2, R3, R4: footprint Resistors_SMD:R_0805 -> Resistor_SMD:R_0805_2012Metric; symbol mb-a-rescue:R-mb-a-rescue -> Device:R
- U2: footprint Housings_SOIC:SOIC-16_3.9x9.9mm_Pitch1.27mm -> Package_SO:SOIC-16_3.9x9.9mm_P1.27mm; symbol mb-a-rescue:PAM8320-mb-a-rescue -> PAM8320:PAM8320
- X1: footprint Connectors:IDC_Header_Straight_6pins -> Connector_IDC:IDC-Header_2x03_P2.54mm_Vertical; symbol mb-a-rescue:I2C-6P-mb-a-rescue -> device.farm:I2C-6P
Connections:
- net +12V: now also C11.2, C4.1, R5.2, U1.5 (VIN)
- net +5V: now also C19.1, L3.2, R6.2
- net GND: now also C11.1, C19.2, C4.2, R7.1, U1.2 (GND)
- new net: C18.1, U1.1 (BST)
- new net: R6.1, R7.2, U1.3 (FB)
- new net: R5.1, U1.4 (SHDN)
- new net: C18.2, L3.1, U1.6 (LX)
Other:
- moved on the sheet: J1, R2, R3, R4, X1
