File: buttons/buttons.kicad_pcb (KiCad board)
At the start: 2 copper layers, 33 x 33 mm, 14 parts, among them J1 GS3, J2 GS3, J3 Buttons, J4 LEDs, U1 STM32F030F4Px, X1 I2C-6P, X2 SWD

Commit message: WIP
Parts:
- added H1: MountingHole, MountingHole:MountingHole_2.2mm_M2, F.Cu at (173.5, 93.0)
- added H2: MountingHole, MountingHole:MountingHole_2.2mm_M2, F.Cu at (173.5, 120.0)
- added H3: MountingHole, MountingHole:MountingHole_2.2mm_M2, F.Cu at (192.5, 93.0)
- added H4: MountingHole, MountingHole:MountingHole_2.2mm_M2, F.Cu at (192.5, 120.0)
- C1, C2, C3: footprint Capacitors_SMD:C_0805 -> Capacitor_SMD:C_0805_2012Metric
- J1, J2: footprint Connectors:GS3 -> Jumper:SolderJumper-3_P1.3mm_Open_Pad1.0x1.5mm
- J3: footprint Pin_Headers:Pin_Header_Straight_2x08_Pitch2.54mm -> Connector_PinHeader_2.54mm:PinHeader_2x08_P2.54mm_Vertical
- J4: footprint Pin_Headers:Pin_Header_Straight_2x04_Pitch2.54mm -> Connector_PinHeader_2.54mm:PinHeader_2x04_P2.54mm_Vertical
- R1, R2, R3, R4: footprint Resistors_SMD:R_0805 -> Resistor_SMD:R_0805_2012Metric
- U1: footprint Housings_SSOP:SSOP-20_4.4x6.5mm_Pitch0.65mm -> Package_SO:SSOP-20_4.4x6.5mm_P0.65mm
- X1: footprint Connectors:IDC_Header_Straight_6pins -> Connector_IDC:IDC-Header_2x03_P2.54mm_Vertical
- moved C2 0.25 mm to (179.0, 109.2)
- turned J1 to 180 degrees
- turned J2 to 180 degrees
- turned X1 to 0 degrees
Routing:
- net (no net): vias 4 -> 0
