File: buttons/buttons.sch (KiCad schematic (older format))
At the start: 14 parts, among them J1 GS3, J2 GS3, J3 Buttons, J4 LEDs, U1 STM32F030F4Px, X1 I2C-6P, X2 SWD

Commit message: WIP
Parts:
- added H1, H2, H3, H4: MountingHole, MountingHole:MountingHole_2.2mm_M2, symbol Mechanical:MountingHole
- C1, C2, C3: footprint Capacitors_SMD:C_0805 -> Capacitor_SMD:C_0805_2012Metric; symbol C -> Device:C
- J1, J2: footprint Connectors:GS3 -> Jumper:SolderJumper-3_P1.3mm_Open_Pad1.0x1.5mm; symbol GS3 -> Jumper:SolderJumper_3_Open
- J3: footprint Pin_Headers:Pin_Header_Straight_2x08_Pitch2.54mm -> Connector_PinHeader_2.54mm:PinHeader_2x08_P2.54mm_Vertical; symbol Conn_02x08_Odd_Even -> Connector_Generic:Conn_02x08_Odd_Even
- J4: footprint Pin_Headers:Pin_Header_Straight_2x04_Pitch2.54mm -> Connector_PinHeader_2.54mm:PinHeader_2x04_P2.54mm_Vertical; symbol Conn_02x04_Odd_Even -> Connector_Generic:Conn_02x04_Odd_Even
- R1, R2, R3, R4: footprint Resistors_SMD:R_0805 -> Resistor_SMD:R_0805_2012Metric; symbol R -> Device:R
- U1: footprint Housings_SSOP:SSOP-20_4.4x6.5mm_Pitch0.65mm -> Package_SO:SSOP-20_4.4x6.5mm_P0.65mm; symbol STM32F030F4Px -> MCU_ST_STM32F0:STM32F030F4Px
- X1: footprint Connectors:IDC_Header_Straight_6pins -> Connector_IDC:IDC-Header_2x03_P2.54mm_Vertical; symbol I2C-6P -> device.farm:I2C-6P
- X2: symbol SWD -> device.farm:SWD
