File: encoder/encoder.sch (KiCad schematic (older format))
At the start: 9 parts, among them J1 GS3, J2 GS3, SW1 Rotary_Encoder_Switch, U1 STM32F030F4Px, X1 I2C-6P, X2 SWD

Commit message: WIP
Parts:
- C1, C2, C3: symbol C -> device:C
- J1, J2: symbol GS3 -> conn:GS3
- SW1: symbol Rotary_Encoder_Switch -> device:Rotary_Encoder_Switch
- U1: symbol STM32F030F4Px -> MCU_ST_STM32F0:STM32F030F4Px
- X1: symbol I2C-6P -> device.farm:I2C-6P
- X2: symbol SWD -> device.farm:SWD
Changed lines of the file:
@@
-EESchema Schematic File Version 2
-LIBS:power
-LIBS:device
-LIBS:switches
-LIBS:relays
-LIBS:motors
-LIBS:transistors
-LIBS:conn
-LIBS:linear
-LIBS:regul
-LIBS:74xx
-LIBS:cmos4000
-LIBS:adc-dac
-LIBS:memory
-LIBS:xilinx
-LIBS:microcontrollers
-LIBS:dsp
-LIBS:microchip
-LIBS:analog_switches
-LIBS:motorola
-LIBS:texas
-LIBS:intel
-LIBS:audio
-LIBS:interface
-LIBS:digital-audio
-LIBS:philips
-LIBS:display
-LIBS:cypress
-LIBS:siliconi
-LIBS:opto
-LIBS:atmel
-LIBS:contrib
-LIBS:valves
-LIBS:device.farm
-LIBS:MCU_ST_STM32F0
+EESchema Schematic File Version 4
 LIBS:encoder-cache
-EELAYER 25 0
+EELAYER 26 0
 EELAYER END
 $Descr A4 11693 8268
@@
 $EndDescr
 $Comp
-L Rotary_Encoder_Switch SW1
+L device:Rotary_Encoder_Switch SW1
 U 1 1 5C2D43A9
 P 6000 3650
@@
 $EndComp
 $Comp
-L I2C-6P X1
+L device.farm:I2C-6P X1
 U 1 1 5C2D4514
 P 2050 3900
@@
 $EndComp
 $Comp
-L STM32F030F4Px U1
+L MCU_ST_STM32F0:STM32F030F4Px U1
 U 1 1 5C2D459B
 P 4450 4050
@@
 SCL
 $Comp
-L +3V3 #PWR01
+L power:+3V3 #PWR01
 U 1 1 5C2D46F6
 P 2400 3700
@@
 NoConn ~ 3950 4350
 $Comp
-L GND #PWR02
+L power:GND #PWR02
 U 1 1 5C2D490B
 P 3950 3750
@@
 $EndComp
 $Comp
-L GND #PWR03
+L power:GND #PWR03
 U 1 1 5C2D491F
 P 4450 4850
@@
 $EndComp
 $Comp
-L C C1
+L device:C C1
 U 1 1 5C2D4945
 P 3700 3550
@@
 $EndComp
 $Comp
-L C C2
+L device:C C2
 U 1 1 5C2D49B4
 P 4250 3200
@@
 $EndComp
 $Comp
-L C C3
+L device:C C3
 U 1 1 5C2D49F5
 P 4750 3200
@@
 	4450 3350 4450 3200
 Wire Wire Line
-	4400 3200 4600 3200
+	4400 3200 4450 3200
 Wire Wire Line
 	4550 3200 4550 3350
@@
 Connection ~ 4500 3200
 $Comp
-L +3V3 #PWR04
+L power:+3V3 #PWR04
 U 1 1 5C2D4A80
 P 4500 3100
@@
 $EndComp
 $Comp
-L GND #PWR05
+L power:GND #PWR05
 U 1 1 5C2D4A9D
 P 4100 3200
@@
 $EndComp
 $Comp
-L GND #PWR06
+L power:GND #PWR06
 U 1 1 5C2D4ABA
 P 4900 3200
@@
 	3850 3550 3950 3550
 $Comp
-L GND #PWR07
+L power:GND #PWR07
 U 1 1 5C2D4AEF
 P 3550 3550
@@
 $EndComp
 $Comp
-L GND #PWR08
+L power:GND #PWR08
 U 1 1 5C2D4B99
 P 6300 3750
@@
 $EndComp
 $Comp
-L GND #PWR09
+L power:GND #PWR09
 U 1 1 5C2D4BB6
 P 5700 3650
@@
 $EndComp
 $Comp
-L GND #PWR010
+L power:GND #PWR010
 U 1 1 5C2D4C2F
 P 2400 4100
@@
 ALERT
 $Comp
-L PWR_FLAG #FLG011
+L power:PWR_FLAG #FLG011
 U 1 1 5C2D4FB2
 P 2250 4700
@@
 $EndComp
 $Comp
-L PWR_FLAG #FLG012
+L power:PWR_FLAG #FLG012
 U 1 1 5C2D4FF2
 P 2250 4800
@@
 $EndComp
 $Comp
-L GND #PWR013
+L power:GND #PWR013
 U 1 1 5C2D500F
 P 2250 4800
@@
 $EndComp
 $Comp
-L +3V3 #PWR014
+L power:+3V3 #PWR014
 U 1 1 5C2D502C
 P 2250 4700
@@
 SWCLK
 $Comp
-L SWD X2
+L device.farm:SWD X2
 U 1 1 5C2D529E
 P 2200 5350
@@
 $EndComp
 $Comp
-L GND #PWR015
+L power:GND #PWR015
 U 1 1 5C2D5329
 P 2550 5350
@@
 SWCLK
 $Comp
-L GS3 J1
+L conn:GS3 J1
 U 1 1 5C2D5CA6
 P 5950 4150
@@
 $EndComp
 $Comp
-L GS3 J2
+L conn:GS3 J2
 U 1 1 5C2D5D1D
 P 5950 4500
@@
 	5250 4500 5800 4500
 $Comp
-L GND #PWR016
+L power:GND #PWR016
 U 1 1 5C2D5F54
 P 6100 4600
@@
 $EndComp
 $Comp
-L GND #PWR017
+L power:GND #PWR017
 U 1 1 5C2D5F7A
 P 6100 4250
@@
 $EndComp
 $Comp
-L +3V3 #PWR018
+L power:+3V3 #PWR018
 U 1 1 5C2D5FA0
 P 6100 4050
@@
 $EndComp
 $Comp
-L +3V3 #PWR019
+L power:+3V3 #PWR019
 U 1 1 5C2D602B
 P 6100 4400
@@
 	0    1    1    0
 $EndComp
+Wire Wire Line
+	4550 3200 4600 3200
+Wire Wire Line
+	4450 3200 4500 3200
+Wire Wire Line
+	4500 3200 4550 3200
 $EndSCHEMATC

Commit message: Band switch support
Parts:
- added H1, H2: MountingHole_Pad, MountingHole:MountingHole_2.2mm_M2_Pad, symbol Mechanical:MountingHole_Pad
- C1, C2, C3: footprint Capacitors_SMD:C_0805 -> Capacitor_SMD:C_0805_2012Metric; symbol device:C -> Device:C
- J1, J2: footprint Connectors:GS3 -> Jumper:SolderJumper-3_P1.3mm_Open_Pad1.0x1.5mm; symbol conn:GS3 -> Jumper:SolderJumper_3_Open
- SW1: footprint Rotary_Encoder:RotaryEncoder_Alps_EC12E-Switch_Vertical_H20mm -> device.farm:RotaryEncoder_Bourns_PEC12R-4x20F-Sxxxx; symbol device:Rotary_Encoder_Switch -> Device:Rotary_Encoder_Switch
- U1: footprint Housings_SSOP:SSOP-20_4.4x6.5mm_Pitch0.65mm -> Package_SO:TSSOP-20_4.4x6.5mm_P0.65mm
- X1: footprint Connectors:IDC_Header_Straight_6pins -> Connector_IDC:IDC-Header_2x03_P2.54mm_Vertical
Connections:
- net GND: now also SW1.C, SW1.S2; no longer SW1.2 (C), SW1.5
- net at U1.6 (PA0): now also SW1.A; no longer SW1.1 (A)
- net at U1.7 (PA1): now also SW1.B; no longer SW1.3 (B)
- net at U1.8 (PA2): now also SW1.S1; no longer SW1.4
Changed lines of the file:
@@
 $EndDescr
 $Comp
-L device:Rotary_Encoder_Switch SW1
+L Device:Rotary_Encoder_Switch SW1
 U 1 1 5C2D43A9
 P 6000 3650
 F 0 "SW1" H 6000 3910 50  0000 C CNN
 F 1 "Rotary_Encoder_Switch" H 6400 3000 50  0001 C CNN
-F 2 "Rotary_Encoder:RotaryEncoder_Alps_EC12E-Switch_Vertical_H20mm" H 5900 3810 50  0001 C CNN
+F 2 "device.farm:RotaryEncoder_Bourns_PEC12R-4x20F-Sxxxx" H 5900 3810 50  0001 C CNN
 F 3 "" H 6000 3910 50  0001 C CNN
 	1    6000 3650
@@
 F 0 "X1" H 2050 4400 60  0000 C CNN
 F 1 "I2C-6P" H 2050 3550 60  0000 C CNN
-F 2 "Connectors:IDC_Header_Straight_6pins" H 2200 4050 60  0001 C CNN
+F 2 "Connector_IDC:IDC-Header_2x03_P2.54mm_Vertical" H 2200 4050 60  0001 C CNN
 F 3 "" H 2200 4050 60  0001 C CNN
 	1    2050 3900
@@
 F 0 "U1" H 4050 4700 50  0000 L CNN
 F 1 "STM32F030F4Px" H 4650 4700 50  0000 L CNN
-F 2 "Housings_SSOP:SSOP-20_4.4x6.5mm_Pitch0.65mm" H 4050 3350 50  0001 R CNN
+F 2 "Package_SO:TSSOP-20_4.4x6.5mm_P0.65mm" H 4050 3350 50  0001 R CNN
 F 3 "" H 4450 4050 50  0001 C CNN
 	1    4450 4050
@@
 $EndComp
 $Comp
-L device:C C1
+L Device:C C1
 U 1 1 5C2D4945
 P 3700 3550
 F 0 "C1" V 3550 3400 50  0000 L CNN
 F 1 "100n" V 3550 3550 50  0000 L CNN
-F 2 "Capacitors_SMD:C_0805" H 3738 3400 50  0001 C CNN
+F 2 "Capacitor_SMD:C_0805_2012Metric" H 3738 3400 50  0001 C CNN
 F 3 "" H 3700 3550 50  0001 C CNN
 	1    3700 3550
@@
 $EndComp
 $Comp
-L device:C C2
+L Device:C C2
 U 1 1 5C2D49B4
 P 4250 3200
 F 0 "C2" V 4100 3050 50  0000 L CNN
 F 1 "100n" V 4100 3200 50  0000 L CNN
-F 2 "Capacitors_SMD:C_0805" H 4288 3050 50  0001 C CNN
+F 2 "Capacitor_SMD:C_0805_2012Metric" H 4288 3050 50  0001 C CNN
 F 3 "" H 4250 3200 50  0001 C CNN
 	1    4250 3200
@@
 $EndComp
 $Comp
-L device:C C3
+L Device:C C3
 U 1 1 5C2D49F5
 P 4750 3200
 F 0 "C3" V 4600 3050 50  0000 L CNN
 F 1 "100n" V 4600 3200 50  0000 L CNN
-F 2 "Capacitors_SMD:C_0805" H 4788 3050 50  0001 C CNN
+F 2 "Capacitor_SMD:C_0805_2012Metric" H 4788 3050 50  0001 C CNN
 F 3 "" H 4750 3200 50  0001 C CNN
 	1    4750 3200
@@
 SWCLK
 $Comp
-L conn:GS3 J1
+L Jumper:SolderJumper_3_Open J1
 U 1 1 5C2D5CA6
-P 5950 4150
-F 0 "J1" H 5600 4150 50  0000 C CNN
-F 1 "GS3" H 5750 4150 50  0000 C CNN
-F 2 "Connectors:GS3" V 6038 4076 50  0001 C CNN
-F 3 "" H 5950 4150 50  0001 C CNN
-	1    5950 4150
+P 5900 4300
+F 0 "J1" H 5750 4250 50  0000 C CNN
+F 1 "GS3" H 5900 4400 50  0000 C CNN
+F 2 "Jumper:SolderJumper-3_P1.3mm_Open_Pad1.0x1.5mm" V 5988 4226 50  0001 C CNN
+F 3 "" H 5900 4300 50  0001 C CNN
+	1    5900 4300
 	-1   0    0    1
 $EndComp
 $Comp
-L conn:GS3 J2
+L Jumper:SolderJumper_3_Open J2
 U 1 1 5C2D5D1D
-P 5950 4500
-F 0 "J2" H 5600 4500 50  0000 C CNN
-F 1 "GS3" H 5750 4500 50  0000 C CNN
-F 2 "Connectors:GS3" V 6038 4426 50  0001 C CNN
-F 3 "" H 5950 4500 50  0001 C CNN
-	1    5950 4500
+P 5900 4650
+F 0 "J2" H 5750 4600 50  0000 C CNN
+F 1 "GS3" H 5900 4750 50  0000 C CNN
+F 2 "Jumper:SolderJumper-3_P1.3mm_Open_Pad1.0x1.5mm" V 5988 4576 50  0001 C CNN
+F 3 "" H 5900 4650 50  0001 C CNN
+	1    5900 4650
 	-1   0    0    1
 $EndComp
@@
 	5300 3850 5300 4150
 Wire Wire Line
-	5300 4150 5800 4150
-Wire Wire Line
 	4950 3950 5250 3950
 Wire Wire Line
 	5250 3950 5250 4500
-Wire Wire Line
-	5250 4500 5800 4500
 $Comp
 L power:GND #PWR016
 U 1 1 5C2D5F54
-P 6100 4600
-F 0 "#PWR016" H 6100 4350 50  0001 C CNN
-F 1 "GND" V 6100 4400 50  0000 C CNN
-F 2 "" H 6100 4600 50  0001 C CNN
-F 3 "" H 6100 4600 50  0001 C CNN
-	1    6100 4600
+P 6100 4300
+F 0 "#PWR016" H 6100 4050 50  0001 C CNN
+F 1 "GND" V 6100 4100 50  0000 C CNN
+F 2 "" H 6100 4300 50  0001 C CNN
+F 3 "" H 6100 4300 50  0001 C CNN
+	1    6100 4300
 	0    -1   -1   0
 $EndComp
@@
 L power:GND #PWR017
 U 1 1 5C2D5F7A
-P 6100 4250
-F 0 "#PWR017" H 6100 4000 50  0001 C CNN
-F 1 "GND" V 6100 4050 50  0000 C CNN
-F 2 "" H 6100 4250 50  0001 C CNN
-F 3 "" H 6100 4250 50  0001 C CNN
-	1    6100 4250
+P 6100 4650
+F 0 "#PWR017" H 6100 4400 50  0001 C CNN
+F 1 "GND" V 6100 4450 50  0000 C CNN
+F 2 "" H 6100 4650 50  0001 C CNN
+F 3 "" H 6100 4650 50  0001 C CNN
+	1    6100 4650
 	0    -1   -1   0
 $EndComp
@@
 L power:+3V3 #PWR018
 U 1 1 5C2D5FA0
-P 6100 4050
-F 0 "#PWR018" H 6100 3900 50  0001 C CNN
-F 1 "+3V3" V 6100 4250 50  0000 C CNN
-F 2 "" H 6100 4050 50  0001 C CNN
-F 3 "" H 6100 4050 50  0001 C CNN
-	1    6100 4050
-	0    1    1    0
+P 5700 4300
+F 0 "#PWR018" H 5700 4150 50  0001 C CNN
+F 1 "+3V3" V 5700 4500 50  0000 C CNN
+F 2 "" H 5700 4300 50  0001 C CNN
+F 3 "" H 5700 4300 50  0001 C CNN
+	1    5700 4300
+	0    -1   -1   0
 $EndComp
 $Comp
 L power:+3V3 #PWR019
 U 1 1 5C2D602B
-P 6100 4400
-F 0 "#PWR019" H 6100 4250 50  0001 C CNN
-F 1 "+3V3" V 6100 4600 50  0000 C CNN
-F 2 "" H 6100 4400 50  0001 C CNN
-F 3 "" H 6100 4400 50  0001 C CNN
-	1    6100 4400
-	0    1    1    0
+P 5700 4650
+F 0 "#PWR019" H 5700 4500 50  0001 C CNN
+F 1 "+3V3" V 5700 4850 50  0000 C CNN
+F 2 "" H 5700 4650 50  0001 C CNN
+F 3 "" H 5700 4650 50  0001 C CNN
+	1    5700 4650
+	0    -1   -1   0
 $EndComp
 Wire Wire Line
@@
 Wire Wire Line
 	4500 3200 4550 3200
+Wire Wire Line
+	5300 4150 5900 4150
+Wire Wire Line
+	5250 4500 5900 4500
+$Comp
+L Mechanical:MountingHole_Pad H2
+U 1 1 5CA2FCA3
+P 7400 3550
+F 0 "H2" H 7500 3601 50  0000 L CNN
+F 1 "MountingHole_Pad" H 7500 3510 50  0000 L CNN
+F 2 "MountingHole:MountingHole_2.2mm_M2_Pad" H 7400 3550 50  0001 C CNN
+F 3 "~" H 7400 3550 50  0001 C CNN
+	1    7400 3550
+	1    0    0    -1
+$EndComp
+$Comp
+L Mechanical:MountingHole_Pad H1
+U 1 1 5CA2FDCD
+P 7400 3300
+F 0 "H1" H 7500 3351 50  0000 L CNN
+F 1 "MountingHole_Pad" H 7500 3260 50  0000 L CNN
+F 2 "MountingHole:MountingHole_2.2mm_M2_Pad" H 7400 3300 50  0001 C CNN
+F 3 "~" H 7400 3300 50  0001 C CNN
+	1    7400 3300
+	1    0    0    -1
+$EndComp
 $EndSCHEMATC
