File: buttons/board/buttons.kicad_pcb (KiCad board)
At the start: 2 copper layers, 31 x 38 mm, 31 parts, among them J1 GS3, J2 GS3, J3 Buttons, J4 LEDs, U1 ATSAMD11D14A-SS, X1 I2C-6P, X2 SWD

Commit message: WIP
Parts:
- C1, C10, C2, C3, C4, C5, C6, C7, C8, C9: footprint Capacitor_SMD:C_0805_2012Metric_Pad1.15x1.40mm_HandSolder -> Capacitor_SMD:C_0805_2012Metric_Pad1.18x1.45mm_HandSolder
- R1, R2, R3, R4: footprint Resistor_SMD:R_0805_2012Metric_Pad1.15x1.40mm_HandSolder -> Resistor_SMD:R_0805_2012Metric_Pad1.20x1.40mm_HandSolder
- R10, R11, R12, R5, R6, R7, R8, R9: value 10k -> 270R; footprint Resistor_SMD:R_0805_2012Metric_Pad1.15x1.40mm_HandSolder -> Resistor_SMD:R_0805_2012Metric_Pad1.20x1.40mm_HandSolder
Connections:
- U1 pad 8: (no net) -> unconnected-(U1-Pad8)
- U1 pad 9: (no net) -> unconnected-(U1-Pad9)
Other:
- net class Default removed
- net class PWR removed
