File: encoder/board/encoder.kicad_pcb (KiCad board)
At the start: 2 copper layers, 32 x 26 mm, 16 parts, among them J1 GS3, J2 GS3, SW1 Rotary_Encoder_Switch, U1 ATSAMD11C14A-SS, X1 I2C-6P, X2 SWD

Commit message: WIP
Parts:
- C1, C2, C3, C4, C5: footprint Capacitor_SMD:C_0805_2012Metric_Pad1.15x1.40mm_HandSolder -> Capacitor_SMD:C_0805_2012Metric_Pad1.18x1.45mm_HandSolder
- R1, R2, R3: footprint Resistor_SMD:R_0805_2012Metric_Pad1.15x1.40mm_HandSolder -> Resistor_SMD:R_0805_2012Metric_Pad1.20x1.40mm_HandSolder
- SW1: value Rotary_Encoder_Switch -> RotaryEncoder_Switch
Connections:
- U1 pad 10: (no net) -> unconnected-(U1-Pad10)
- X1 pad 5: (no net) -> unconnected-(X1-Pad5)
Other:
- net class Default removed
